Commit message: Add Gazebo launch file and update URDF for right wheel material

File: description/common.urdf.xacro (robot description, xacro)
@@ -132,4 +132,7 @@
         </xacro:inertial_cylinder>
     </link>
+     <gazebo reference="right_wheel">
+        <material>Gazebo/Blue</material>
+    </gazebo>
     <!-- BÁNH HƯỚNG TRƯỚC (FRONT CASTER WHEEL) -->
     <joint name="front_caster_wheel_joint" type="fixed">

Commit message: Add files via upload

File: description/common.urdf.xacro (robot description, xacro)
@@ -86,4 +86,8 @@
         </xacro:inertial_cylinder>
     </link>
+    <!--
+    <gazebo reference="chassis">
+        <material>Gazebo/White</material>
+    </gazebo> -->
     <!-- BÁNH TRÁI (LEFT WHEEL) -->
     <joint name="left_wheel_joint" type="continuous">
@@ -109,4 +113,7 @@
         </xacro:inertial_cylinder>
     </link>
+    <!-- <gazebo reference="left_wheel">
+        <material>Gazebo/Blue</material>
+    </gazebo> -->
     <!-- BÁNH PHẢI (RIGHT WHEEL) -->
     <joint name="right_wheel_joint" type="continuous">
@@ -132,12 +139,12 @@
         </xacro:inertial_cylinder>
     </link>
-     <gazebo reference="right_wheel">
+     <!-- <gazebo reference="right_wheel">
         <material>Gazebo/Blue</material>
-    </gazebo>
+    </gazebo> -->
     <!-- BÁNH HƯỚNG TRƯỚC (FRONT CASTER WHEEL) -->
     <joint name="front_caster_wheel_joint" type="fixed">
         <parent link="chassis"/>
         <child link="front_caster_wheel"/>
-        <origin xyz="0.16 0 -0.01" rpy="0 0 0"/>
+        <origin xyz="0.16 0 -0.045" rpy="0 0 0"/>
     </joint>
     <link name="front_caster_wheel">
@@ -157,9 +164,14 @@
         </xacro:inertial_sphere>
     </link>
+    <!-- <gazebo reference="front_caster_wheel">
+        <material>Gazebo/Black</material>
+        <mu1 value="0.001"/>
+        <mu2 value="0.001"/>
+    </gazebo> -->
     <!-- BÁNH HƯỚNG SAU (REAR CASTER WHEEL) -->
     <joint name="rear_caster_wheel_joint" type="fixed">
         <parent link="chassis"/>
         <child link="rear_caster_wheel"/>
-        <origin xyz="-0.16 0 -0.01" rpy="0 0 0"/>
+        <origin xyz="-0.16 0 -0.045" rpy="0 0 0"/>
     </joint>
     <link name="rear_caster_wheel">
@@ -179,3 +191,8 @@
         </xacro:inertial_sphere>
     </link>
+     <!-- <gazebo reference="rear_caster_wheel">
+        <material>Gazebo/Black</material>
+        <mu1 value="0.001"/>
+        <mu2 value="0.001"/>
+    </gazebo> -->
 </robot>

File: description/robot.urdf.xacro (robot description, xacro)
@@ -1,4 +1,9 @@
 <?xml version="1.0"?>
 <robot xmlns:xacro="http://www.ros.org/wiki/xacro"  name="robot">
+   <xacro:arg name="use_ros2_control" default="true"/>
+    <xacro:arg name="sim_mode" default="false"/>
    <xacro:include filename="common.urdf.xacro"/>
+   <!-- <xacro:include filename="gazebo_control.xacro" /> -->
+    <xacro:include filename="ros2Control.xacro" />
+   <!-- <xacro:include filename="lidar.xacro" /> -->
 </robot>
