Commit message: Add files via upload

File: description/lidar.xacro (robot description, xacro)
@@ -22,32 +22,3 @@
         </xacro:inertial_cylinder>
     </link>
-<!--
-    <gazebo reference="laser_frame">
-        <material>Gazebo/Red</material>
-        <sensor name="laser" type="ray">
-            <pose> 0 0 0 0 0 0 </pose>
-            <visualize>true</visualize>
-            <update_rate>10</update_rate>
-            <ray>
-                <scan>
-                    <horizontal>
-                        <samples>360</samples>
-                        <min_angle>-3.14</min_angle>
-                        <max_angle>3.14</max_angle>
-                    </horizontal>
-                </scan>
-                <range>
-                    <min>0.3</min>
-                    <max>12</max>
-                </range>
-            </ray>
-            <plugin name="laser_controller" filename="libgazebo_ros_ray_sensor.so">
-                <ros>
-                    <argument>~/out:=scan</argument>
-                </ros>
-                <output_type>sensor_msgs/LaserScan</output_type>
-                <frame_name>laser_frame</frame_name>
-            </plugin>
-        </sensor>
-    </gazebo> -->
 </robot>

File: description/robot.urdf.xacro (robot description, xacro)
@@ -4,6 +4,5 @@
     <xacro:arg name="sim_mode" default="false"/>
    <xacro:include filename="common.urdf.xacro"/>
-   <!-- <xacro:include filename="gazebo_control.xacro" /> -->
-    <xacro:include filename="ros2Control.xacro" />
-   <!-- <xacro:include filename="lidar.xacro" /> -->
+   <xacro:include filename="ros2Control.xacro" />
+   <xacro:include filename="$(find eddie_bot)/description/lidar.xacro" />
 </robot>
